File: minitiouner-rt5047.kicad_pcb (KiCad board)
At the start: 2 copper layers, 99.9 x 47 mm, 27 parts, among them IC1 TLV76033, IC2 RT5047A

Commit message: WIP
Parts:
- added J1: CONN_01x02, Connector_Molex:Molex_KK-254_AE-6410-02A_1x02_P2.54mm_Vertical, F.Cu at (46.7, 116.8)
- added J2: A_LNB_POWER, Connector_Molex:Molex_KK-254_AE-6410-02A_1x02_P2.54mm_Vertical, F.Cu at (56.1, 117.0)
- added J3: A_FAULT_LED, Connector_Molex:Molex_KK-254_AE-6410-02A_1x02_P2.54mm_Vertical, F.Cu at (91.6, 116.8)
- added J4: A_SEL_SWITCH, Connector_Molex:Molex_KK-254_AE-6410-03A_1x03_P2.54mm_Vertical, F.Cu at (99.3, 116.8)
- added J5: CONN_01x04, Connector_Molex:Molex_KK-254_AE-6410-04A_1x04_P2.54mm_Vertical, F.Cu at (127.0, 117.2)
- added L1: 10u, agg:1210, F.Cu at (62.2, 97.8)
- added Q1: BC817, Package_TO_SOT_SMD:SOT-23, F.Cu at (89.4, 110.5)
- added R6: 47R, agg:0603, F.Cu at (94.0, 110.5)
- moved C1 72.6 mm to (76.2, 115.6), turned to 180 degrees
- moved C7 69.0 mm to (56.2, 107.8), turned to 180 degrees
- moved FB2 66.3 mm to (58.7, 109.6), turned to 90 degrees
- moved C10 63.8 mm to (48.6, 96.0)
- moved C12 63.8 mm to (57.5, 112.1), turned to 180 degrees
- moved IC1 61.2 mm to (76.2, 111.9)
- moved C8 59.1 mm to (56.3, 103.9), turned to 180 degrees
- moved C9 56.3 mm to (76.1, 108.5)
- moved C6 56.2 mm to (48.6, 98.6)
- moved FB1 54.0 mm to (58.7, 106.2), turned to 90 degrees
- moved C3 50.6 mm to (55.4, 86.7), turned to 270 degrees
- moved D3 49.1 mm to (62.2, 92.7)
- moved R2 48.5 mm to (80.0, 94.0), turned to 180 degrees
- moved C5 48.3 mm to (47.9, 86.4), turned to 270 degrees
- moved R3 48.3 mm to (78.7, 100.3), turned to 180 degrees
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Connections:
- R3 pad 1: 3v3 -> A_TONE_PIN
- R3 pad 2: A_TONE_PIN -> GND

Commit message: WIP.
Parts:
- added C13: 10n, agg:0603, F.Cu at (65.2, 109.3)
- added C14: 10n, agg:0603, F.Cu at (65.0, 112.3)
- added C15: 100n, agg:0603, F.Cu at (48.9, 105.9)
- added C16: 100n, agg:0603, F.Cu at (65.1, 106.3)
- added C17: 100n, agg:0603, F.Cu at (56.2, 106.2)
- added C18: 100n, agg:0603, F.Cu at (111.1, 116.2)
- added C19: 100n, agg:0603, F.Cu at (101.2, 116.2)
- added C20: 100n, agg:0603, F.Cu at (120.8, 116.2)
- added FB3: Ferrite_Bead_Small, agg:0805, F.Cu at (68.1, 107.3)
- added FB4: Ferrite_Bead_Small, agg:0805, F.Cu at (68.1, 111.4)
- added FB5: Ferrite_Bead_Small, agg:0805, F.Cu at (50.1, 109.4)
- added J6: B_LNB_POWER, Connector_Molex:Molex_KK-254_AE-6410-02A_1x02_P2.54mm_Vertical, F.Cu at (65.3, 116.6)
- added J7: TONE_SWITCH, Connector_Molex:Molex_KK-254_AE-6410-02A_1x02_P2.54mm_Vertical, F.Cu at (105.6, 116.2)
- added JP3: SEL_REMOTE, Jumper:SolderJumper-2_P1.3mm_Open_Pad1.0x1.5mm, F.Cu at (128.7, 106.0)
- added R7: 4K7, agg:0603, F.Cu at (124.5, 101.0)
- D2, D3, D4: footprint agg:SOD-123 -> agg:DO-214AC-SMA
- FB1, FB2: footprint agg:0603 -> agg:0805
- J1: value CONN_01x02 -> 12V_INPUT
- J3: value A_FAULT_LED -> FAULT_LED
- J4: value A_SEL_SWITCH -> VSEL_SWITCH
- J5: value CONN_01x04 -> USB_CONTROL
- JP1: value A_EN_REMOTE_JMP -> EN_REMOTE; footprint Jumper:SolderJumper-3_P1.3mm_Open_RoundedPad1.0x1.5mm -> Jumper:SolderJumper-2_P1.3mm_Open_Pad1.0x1.5mm
- JP2: value A_TONE_REMOTE_JMP -> TONE_REMOTE; footprint Jumper:SolderJumper-3_P1.3mm_Open_RoundedPad1.0x1.5mm -> Jumper:SolderJumper-2_P1.3mm_Open_Pad1.0x1.5mm
- L1: footprint agg:1210 -> Inductor_SMD:L_Bourns_SRN6045TA
- moved JP1 58.3 mm to (132.9, 106.0), turned to 270 degrees
- moved JP2 48.0 mm to (124.5, 106.0), turned to 270 degrees
- moved R5 41.7 mm to (128.7, 101.0)
- moved Q1 24.9 mm to (114.3, 110.2)
- moved R6 23.9 mm to (117.9, 109.7)
- moved J3 23.8 mm to (115.3, 116.2)
- moved C10 20.7 mm to (68.3, 102.4)
- moved C6 19.7 mm to (68.3, 100.3)
- moved C8 18.2 mm to (68.8, 90.7), turned to 270 degrees
- moved R1 15.8 mm to (95.8, 90.8), turned to 270 degrees
- moved C2 15.6 mm to (65.2, 91.4), turned to 90 degrees
- moved R2 14.3 mm to (93.9, 90.8), turned to 270 degrees
- moved R3 13.3 mm to (92.0, 99.3), turned to 270 degrees
- moved C5 12.3 mm to (59.1, 91.4), turned to 90 degrees
- moved R4 12.2 mm to (92.0, 90.8), turned to 270 degrees
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Connections:
- C12 pad 2: Net-(C12-Pad2) -> GND
- C7 pad 2: Net-(C12-Pad2) -> GND
- IC2 pad 5: A_TONE_PIN -> A_EN_PIN
- IC2 pad 6: A_FAULT_PIN -> A_SEL_PIN
- IC2 pad 7: A_SEL_PIN -> A_FAULT_PIN
- IC2 pad 8: A_EN_PIN -> A_TONE_PIN
- J1 pad 1: Net-(C1-Pad2) -> GND
- J1 pad 2: GND -> Net-(FB5-Pad2)
- J2 pad 1: Net-(C12-Pad2) -> GND
- JP2 pad 1: A_TONE_PIN -> Net-(JP2-Pad1)
- R5 pad 1: A_SEL_REMOTE -> Net-(JP3-Pad1)
Routing:
- net GND: track 0.00 -> 227.2 mm, vias 0 -> 12
- net 3v3: track 0.00 -> 103.0 mm, vias 0 -> 2
- net A_SEL_PIN: track 0.00 -> 85.3 mm, vias 0 -> 5
- net A_TONE_PIN: track 0.00 -> 76.7 mm, vias 0 -> 3
- net A_EN_PIN: track 0.00 -> 71.9 mm, vias 0 -> 2
- net Net-(C1-Pad2): track 0.00 -> 70.5 mm, vias 0 -> 2
- net Net-(C16-Pad1): track 0.00 -> 65.5 mm
- net A_FAULT_PIN: track 0.00 -> 55.5 mm, vias 0 -> 4
- net Net-(C2-Pad1): track 0.00 -> 27.0 mm
- net A_TONE_REMOTE: track 0.00 -> 10.9 mm
- net Net-(D3-Pad2): track 0.00 -> 10.7 mm
- net A_SEL_REMOTE: track 0.00 -> 10.2 mm
- net A_EN_REMOTE: track 0.00 -> 9.51 mm
- net Net-(C12-Pad1): track 0.00 -> 6.80 mm
- net Net-(C14-Pad1): track 0.00 -> 6.66 mm
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- added copper zone on B.Cu, net GND
- added copper zone on F.Cu, net GND
Other:
- board text added: "Input: 8V - 16V"
- board text added: "Minitiouner LNB Power Supply"
- board text added: "Output: 13.3V / 18.3V"
- board text added: "Phil M0DNY"
- board text added: "r2019.08"
