File: minitiouner-rt5047.sch (KiCad schematic (older format))
At the start: 14 parts

Commit message: WIP.
Parts:
- removed C? (x2): 10u, symbol agg-kicad:C
- removed C?: 1u, symbol agg-kicad:C
- removed D? (x2): SS14, symbol agg-kicad:SCHOTTKY
- removed IC?: RT5047A, agg:SOIC-8-EP, symbol agg-kicad:RT5047A
- removed L?: 10u, symbol agg-kicad:L
- added C1, C8, C9: 100n, agg:0603, symbol agg-kicad:C
- added C12, C7: 10n, agg:0603, symbol agg-kicad:C
- added C2, C3, C4, C5: 10u, agg:0805, symbol agg-kicad:C
- added D1: SMDJ20A, agg:DO-214AB-SMC, symbol agg-kicad:SCHOTTKY
- added D2: SS14, agg:SOD-123, symbol agg-kicad:SCHOTTKY
- added FB1, FB2: Ferrite_Bead_Small, agg:0603, symbol Device:Ferrite_Bead_Small
- added IC1: TLV76033, agg:SOT-23, symbol agg-kicad:TLV76033
- added J1: CONN_01x02, symbol agg-kicad:CONN_01x02
- added J2: A_LNB_POWER, symbol agg-kicad:CONN_01x02
- added J3: A_FAULT_LED, symbol agg-kicad:CONN_01x02
- added J4: A_SEL_SWITCH, symbol agg-kicad:CONN_01x03
- added J5: CONN_01x04, symbol agg-kicad:CONN_01x04
- added JP1: A_EN_REMOTE_JMP, Jumper:SolderJumper-3_P1.3mm_Open_RoundedPad1.0x1.5mm, symbol Jumper:SolderJumper_2_Open
- added JP2: A_TONE_REMOTE_JMP, Jumper:SolderJumper-3_P1.3mm_Open_RoundedPad1.0x1.5mm, symbol Jumper:SolderJumper_2_Open
- added R1, R2, R3: 47K, agg:0603, symbol agg-kicad:R
- added R4, R5: 4K7, agg:0603, symbol agg-kicad:R
- C10, C6: renamed from C?; footprint (none) -> agg:0805
- C11: renamed from C?; footprint (none) -> agg:0603
- D3, D4: renamed from D?; footprint (none) -> agg:SOD-123
- gave numbers to parts that had none: 2
Connections:
- net at IC2.1 (LNB): now also D4.2, C8.1, D1.1, D2.1, FB1.2
- net at IC2.2 (BOOST): now also D3.1, D4.1, C2.1, C3.1, C4.1, C5.1
- net at IC2.3 (LX): now also D3.2, L1.2
- net at IC2.4 (VIN): now also C10.1, C11.1, C6.1, L1.1, C1.2, IC1.2 (VIN), J1.1
- net A_EN_PIN: now reaches IC2.5 (EN)
- net A_EN_PIN: now also JP1.1 (A), R1.2
- net A_SEL_PIN: now reaches IC2.6 (SEL)
- net A_SEL_PIN: now also J4.2, R2.2, R5.2
- net A_FAULT_PIN: now reaches IC2.7 (FAULT)
- net A_FAULT_PIN: now also J3.2, R4.2
- net A_TONE_PIN: now reaches IC2.8 (TONE)
- net A_TONE_PIN: now also JP2.1 (A), R3.2
- net GND: now reaches IC2.EP (GND)
- net GND: now also C10.2, C11.2, C6.2, C1.1, C2.2, C3.2, C4.2, C5.2, C8.2, C9.2, D1.2, D2.2, IC1.3 (GND), J1.2, J3.1, J4.1, J5.1
- new net: C7.1, FB1.1, FB2.2
- new net: C12.2, C7.2, J2.1
- new net: C12.1, FB2.1, J2.2
- new net 3v3: C9.1, IC1.1 (VOUT), J4.3, R1.1, R2.1, R3.1, R4.1
- new net A_EN_REMOTE: J5.4, JP1.2 (B)
- new net A_SEL_REMOTE: J5.3, R5.1
- new net A_TONE_REMOTE: J5.2, JP2.2 (B)
Other:
- note added: "700KHz F_Sw"
- note added: "LED I = 0.5mA"
- moved on the sheet: C10, C6, D3, D4, L1

Commit message: WIP
Parts:
- added Q1: BC817, Package_TO_SOT_SMD:SOT-23, symbol Transistor_BJT:BC817
- added R6: 47R, agg:0603, symbol agg-kicad:R
- IC2: symbol agg-kicad:RT5047A -> minitiouner-rt5047-rescue:RT5047A-agg-kicad
- J1, J2, J3: footprint (none) -> Connector_Molex:Molex_KK-254_AE-6410-02A_1x02_P2.54mm_Vertical
- J4: footprint (none) -> Connector_Molex:Molex_KK-254_AE-6410-03A_1x03_P2.54mm_Vertical
- J5: footprint (none) -> Connector_Molex:Molex_KK-254_AE-6410-04A_1x04_P2.54mm_Vertical
- L1: footprint (none) -> agg:1210
Connections:
- net 3v3: now also R6.2; no longer R3.1
- net A_EN_PIN: now also IC2.8 (EN); no longer IC2.5 (EN)
- net A_FAULT_PIN: now also IC2.6 (FAULT), Q1.1 (B); no longer IC2.7 (FAULT), J3.2
- net A_SEL_PIN: now also IC2.7 (SEL); no longer IC2.6 (SEL)
- net A_TONE_PIN: now also IC2.5 (TONE), R3.1; no longer IC2.8 (TONE), R3.2
- net GND: now also R3.2, Q1.2 (E); no longer J3.1
- new net: J3.1, Q1.3 (C)
- new net: J3.2, R6.1
Other:
- note added: "Default: 18V"
- note added: "Default: Enable ON"
- note added: "Default: Tone OFF"
- note added: "Driver I = 0.5mA"
- note removed: "LED I = 0.5mA"
- moved on the sheet: J3, R3
Changed lines of the file:
@@
 $EndDescr
 $Comp
-L agg-kicad:RT5047A IC2
+L minitiouner-rt5047-rescue:RT5047A-agg-kicad IC2
 U 1 1 5D5C8177
 P 3750 3350
@@
 F 0 "L1" H 2900 3531 50  0000 C CNN
 F 1 "10u" H 2900 3440 50  0000 C CNN
-F 2 "" H 2850 3350 50  0001 C CNN
+F 2 "agg:1210" H 2850 3350 50  0001 C CNN
 F 3 "" H 2850 3350 50  0001 C CNN
 	1    2850 3350
@@
 	0    1    1    0
 $EndComp
-Wire Wire Line
-	5000 5350 5000 5250
-Connection ~ 5000 5350
-Text Notes 5250 5550 0    50   ~ 0
-LED I = 0.5mA
+Text Notes 4800 5450 0    50   ~ 0
+Driver I = 0.5mA
 $Comp
 L Jumper:SolderJumper_2_Open JP2
@@
 F 0 "J5" H 8672 4199 50  0000 R CNN
 F 1 "CONN_01x04" H 8672 4290 50  0000 R CNN
-F 2 "" H 8750 4400 50  0001 C CNN
+F 2 "Connector_Molex:Molex_KK-254_AE-6410-04A_1x04_P2.54mm_Vertical" H 8750 4400 50  0001 C CNN
 F 3 "" H 8750 4400 50  0001 C CNN
 	1    8750 4400
@@
 F 0 "J1" H 1633 3665 50  0000 C CNN
 F 1 "CONN_01x02" H 1633 3574 50  0000 C CNN
-F 2 "" H 1600 3450 50  0001 C CNN
+F 2 "Connector_Molex:Molex_KK-254_AE-6410-02A_1x02_P2.54mm_Vertical" H 1600 3450 50  0001 C CNN
 F 3 "" H 1600 3450 50  0001 C CNN
 	1    1600 3450
@@
 F 0 "J4" H 5522 4649 50  0000 R CNN
 F 1 "A_SEL_SWITCH" H 5522 4740 50  0000 R CNN
-F 2 "" H 5600 4800 50  0001 C CNN
+F 2 "Connector_Molex:Molex_KK-254_AE-6410-03A_1x03_P2.54mm_Vertical" H 5600 4800 50  0001 C CNN
 F 3 "" H 5600 4800 50  0001 C CNN
 	1    5600 4800
@@
 F 0 "J2" H 3672 2649 50  0000 R CNN
 F 1 "A_LNB_POWER" H 3672 2740 50  0000 R CNN
-F 2 "" H 3750 2750 50  0001 C CNN
+F 2 "Connector_Molex:Molex_KK-254_AE-6410-02A_1x02_P2.54mm_Vertical" H 3750 2750 50  0001 C CNN
 F 3 "" H 3750 2750 50  0001 C CNN
 	1    3750 2750
@@
 L agg-kicad:CONN_01x02 J3
 U 1 1 5D7F60CC
-P 5200 5450
-F 0 "J3" H 5122 5349 50  0000 R CNN
-F 1 "A_FAULT_LED" H 5122 5440 50  0000 R CNN
-F 2 "" H 5200 5450 50  0001 C CNN
-F 3 "" H 5200 5450 50  0001 C CNN
-	1    5200 5450
+P 6350 5100
+F 0 "J3" H 6272 4999 50  0000 R CNN
+F 1 "A_FAULT_LED" H 6272 5090 50  0000 R CNN
+F 2 "Connector_Molex:Molex_KK-254_AE-6410-02A_1x02_P2.54mm_Vertical" H 6350 5100 50  0001 C CNN
+F 3 "" H 6350 5100 50  0001 C CNN
+	1    6350 5100
 	-1   0    0    1
 $EndComp
-Wire Wire Line
-	5000 5350 5100 5350
 $Comp
 L agg-kicad:GND #PWR0107
 U 1 1 5D7FCB47
-P 5000 5500
-F 0 "#PWR0107" H 4870 5540 50  0001 L CNN
-F 1 "GND" H 5000 5589 50  0000 C CNN
-F 2 "" H 5000 5500 50  0001 C CNN
-F 3 "" H 5000 5500 50  0001 C CNN
-	1    5000 5500
-	1    0    0    -1
-$EndComp
-Wire Wire Line
-	5000 5500 5000 5450
-Wire Wire Line
-	5000 5450 5100 5450
+P 6200 5650
+F 0 "#PWR0107" H 6070 5690 50  0001 L CNN
+F 1 "GND" H 6200 5739 50  0000 C CNN
+F 2 "" H 6200 5650 50  0001 C CNN
+F 3 "" H 6200 5650 50  0001 C CNN
+	1    6200 5650
+	1    0    0    -1
+$EndComp
 $Comp
 L agg-kicad:GND #PWR0108
@@
 L agg-kicad:R R3
 U 1 1 5D820FB9
-P 4900 5850
-F 0 "R3" V 4904 5894 50  0000 L CNN
-F 1 "47K" V 4995 5894 50  0000 L CNN
-F 2 "agg:0603" H 4900 5850 50  0001 C CNN
-F 3 "" H 4900 5850 50  0001 C CNN
-	1    4900 5850
+P 4900 6100
+F 0 "R3" V 4904 6144 50  0000 L CNN
+F 1 "47K" V 4995 6144 50  0000 L CNN
+F 2 "agg:0603" H 4900 6100 50  0001 C CNN
+F 3 "" H 4900 6100 50  0001 C CNN
+	1    4900 6100
 	0    1    1    0
 $EndComp
@@
 Text GLabel 4750 6000 0    50   Input ~ 0
 A_TONE_PIN
-Wire Wire Line
-	4750 6000 4900 6000
-Wire Wire Line
-	4900 6000 4900 5950
-$Comp
-L agg-kicad:3v3 #PWR0109
-U 1 1 5D82F1E0
-P 4900 5800
-F 0 "#PWR0109" H 4900 5910 50  0001 L CNN
-F 1 "3v3" H 4900 5923 50  0000 C CNN
-F 2 "" H 4900 5800 50  0001 C CNN
-F 3 "" H 4900 5800 50  0001 C CNN
-	1    4900 5800
-	1    0    0    -1
-$EndComp
-Wire Wire Line
-	4900 5800 4900 5850
 Text GLabel 4750 5350 0    50   Input ~ 0
 A_FAULT_PIN
@@
 Wire Wire Line
 	4150 3350 4250 3350
-Wire Wire Line
-	5350 6000 4900 6000
-Connection ~ 4900 6000
 Text GLabel 4700 3950 0    50   Input ~ 0
 A_EN_PIN
@@
 Wire Wire Line
 	8650 4300 8350 4300
+$Comp
+L Transistor_BJT:BC817 Q1
+U 1 1 5D768D02
+P 6100 5350
+F 0 "Q1" H 6291 5396 50  0000 L CNN
+F 1 "BC817" H 6291 5305 50  0000 L CNN
+F 2 "Package_TO_SOT_SMD:SOT-23" H 6300 5275 50  0001 L CIN
+F 3 "http://www.fairchildsemi.com/ds/BC/BC817.pdf" H 6100 5350 50  0001 L CNN
+F 4 "1902482" H 6100 5350 50  0001 C CNN "FARNELL"
+	1    6100 5350
+	1    0    0    -1
+$EndComp
+$Comp
+L agg-kicad:R R6
+U 1 1 5D76DC55
+P 6150 5000
+F 0 "R6" V 6154 5044 50  0000 L CNN
+F 1 "47R" V 6245 5044 50  0000 L CNN
+F 2 "agg:0603" H 6150 5000 50  0001 C CNN
+F 3 "" H 6150 5000 50  0001 C CNN
+	1    6150 5000
+	-1   0    0    1
+$EndComp
+$Comp
+L agg-kicad:3v3 #PWR0109
+U 1 1 5D76E22B
+P 6000 4950
+F 0 "#PWR0109" H 6000 5060 50  0001 L CNN
+F 1 "3v3" H 6000 5073 50  0000 C CNN
+F 2 "" H 6000 4950 50  0001 C CNN
+F 3 "" H 6000 4950 50  0001 C CNN
+	1    6000 4950
+	1    0    0    -1
+$EndComp
+$Comp
+L agg-kicad:GND #PWR0111
+U 1 1 5D772B42
+P 4900 6300
+F 0 "#PWR0111" H 4770 6340 50  0001 L CNN
+F 1 "GND" H 4900 6389 50  0000 C CNN
+F 2 "" H 4900 6300 50  0001 C CNN
+F 3 "" H 4900 6300 50  0001 C CNN
+	1    4900 6300
+	1    0    0    -1
+$EndComp
+Wire Wire Line
+	4750 6000 4900 6000
+Wire Wire Line
+	4900 6100 4900 6000
+Connection ~ 4900 6000
+Wire Wire Line
+	4900 6000 5350 6000
+Wire Wire Line
+	4900 6200 4900 6300
+Text Notes 4650 6450 0    50   ~ 0
+Default: Tone OFF
+Text Notes 4350 4100 0    50   ~ 0
+Default: Enable ON
+Text Notes 4300 4850 0    50   ~ 0
+Default: 18V
+Wire Wire Line
+	6200 5550 6200 5650
+Wire Wire Line
+	6250 5100 6200 5100
+Wire Wire Line
+	6200 5100 6200 5150
+Wire Wire Line
+	5000 5250 5000 5350
+Wire Wire Line
+	5900 5350 5000 5350
+Connection ~ 5000 5350
+Wire Wire Line
+	6150 5000 6250 5000
+Wire Wire Line
+	6050 5000 6000 5000
+Wire Wire Line
+	6000 5000 6000 4950
 $EndSCHEMATC

Commit message: WIP.
Parts:
- added C13, C14: 10n, agg:0603, symbol agg-kicad:C
- added C15, C16, C17, C18, C19, C20: 100n, agg:0603, symbol agg-kicad:C
- added FB3, FB4, FB5: Ferrite_Bead_Small, agg:0805, symbol Device:Ferrite_Bead_Small
- added J6: B_LNB_POWER, Connector_Molex:Molex_KK-254_AE-6410-02A_1x02_P2.54mm_Vertical, symbol agg-kicad:CONN_01x02
- added J7: TONE_SWITCH, Connector_Molex:Molex_KK-254_AE-6410-02A_1x02_P2.54mm_Vertical, symbol agg-kicad:CONN_01x02
- added JP3: SEL_REMOTE, Jumper:SolderJumper-2_P1.3mm_Open_Pad1.0x1.5mm, symbol Jumper:SolderJumper_2_Open
- added R7: 4K7, agg:0603, symbol agg-kicad:R
- D2, D3, D4: footprint agg:SOD-123 -> agg:DO-214AC-SMA
- FB1, FB2: footprint agg:0603 -> agg:0805; FARNELL (none) -> 2859031
- IC2: symbol minitiouner-rt5047-rescue:RT5047A-agg-kicad -> agg-kicad:RT5047A
- J1: value CONN_01x02 -> 12V_INPUT
- J3: value A_FAULT_LED -> FAULT_LED
- J4: value A_SEL_SWITCH -> VSEL_SWITCH
- J5: value CONN_01x04 -> USB_CONTROL
- JP1: value A_EN_REMOTE_JMP -> EN_REMOTE; footprint Jumper:SolderJumper-3_P1.3mm_Open_RoundedPad1.0x1.5mm -> Jumper:SolderJumper-2_P1.3mm_Open_Pad1.0x1.5mm
- JP2: value A_TONE_REMOTE_JMP -> TONE_REMOTE; footprint Jumper:SolderJumper-3_P1.3mm_Open_RoundedPad1.0x1.5mm -> Jumper:SolderJumper-2_P1.3mm_Open_Pad1.0x1.5mm
- L1: footprint agg:1210 -> Inductor_SMD:L_Bourns_SRN6045TA; FARNELL (none) -> 2061652
Connections:
- net 3v3: now also C18.1, C19.1, C20.1, J7.2
- net A_EN_PIN: now also IC2.5 (EN); no longer IC2.8 (EN)
- net A_FAULT_PIN: now also IC2.7 (FAULT); no longer IC2.6 (FAULT)
- net A_SEL_PIN: now also IC2.6 (SEL); no longer IC2.7 (SEL)
- net A_SEL_REMOTE: now also JP3.2 (B); no longer R5.1
- net A_TONE_PIN: now also IC2.8 (TONE), J7.1, R7.2; no longer IC2.5 (TONE), JP2.1 (A)
- net GND: now also C12.2, C7.2, J1.1, J2.1, C13.2, C14.2, C15.2, C16.2, C17.2, C18.2, C19.2, C20.2, J6.1; no longer J1.2
- net at C8.1, D1.1, D2.1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: now also C16.1, C17.1, FB3.2
- net at C1.2, C10.1, C11.1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: now also C15.1, FB5.1; no longer J1.1
- new net: JP2.1 (A), R7.1
- new net: FB5.2, J1.2
- new net: JP3.1 (A), R5.1
- new net: C13.1, FB3.1, FB4.2
- new net: C14.1, FB4.1, J6.2
Other:
- moved on the sheet: J1, JP2
